File: pga2311.kicad_pcb (KiCad board)
At the start: 2 copper layers, 50 x 50 mm, 26 parts, among them P1 VIN_R, P2 VOUT_R, P3 VIN_L, P4 VOUT_L, P6 SDO_TO_OTHER_PGA2311, U1 PGA2311

Commit message: before making changes
Changed lines of the file:
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@@
-(kicad_pcb (version 4) (host pcbnew 0.201508170901+6097~28~ubuntu14.04.1-product)
+(kicad_pcb (version 4) (host pcbnew 0.201601191446+6495~42~ubuntu15.10.1-product)
   (general
     (links 43)
@@
     (area 48.115999 32.857999 98.216001 82.958001)
     (thickness 1.6)
-    (drawings 75)
+    (drawings 83)
     (tracks 150)
     (zones 0)
@@
     (at 50.2 58.2 90)
     (descr "JST PH series connector, B5B-PH-KL")
-    (fp_text reference P5 (at 0 -2.99974 90) (layer F.SilkS)
+    (fp_text reference P5 (at 0 -2.99974 90) (layer F.SilkS) hide
       (effects (font (thickness 0.3048)))
     )
@@
     (descr "Terminal block 2 pins")
     (tags DEV)
-    (fp_text reference P1 (at 0 -5.842) (layer F.SilkS)
+    (fp_text reference P1 (at 0 -5.842) (layer F.SilkS) hide
       (effects (font (thickness 0.3048)))
     )
@@
     (descr "Terminal block 2 pins")
     (tags DEV)
-    (fp_text reference P2 (at 0 -5.842 180) (layer F.SilkS)
+    (fp_text reference P2 (at 0 -5.842 180) (layer F.SilkS) hide
       (effects (font (thickness 0.3048)))
     )
@@
     (descr "Terminal block 2 pins")
     (tags DEV)
-    (fp_text reference P3 (at 0 -5.842) (layer F.SilkS)
+    (fp_text reference P3 (at 0 -5.842) (layer F.SilkS) hide
       (effects (font (thickness 0.3048)))
     )
@@
     (descr "Terminal block 2 pins")
     (tags DEV)
-    (fp_text reference P4 (at 0 -5.842 180) (layer F.SilkS)
+    (fp_text reference P4 (at 0 -5.842 180) (layer F.SilkS) hide
       (effects (font (thickness 0.3048)))
     )
@@
     (descr "Terminal block 2 pins")
     (tags DEV)
-    (fp_text reference P8 (at 0 -5.842 90) (layer F.SilkS)
+    (fp_text reference P8 (at 0 -5.842 90) (layer F.SilkS) hide
       (effects (font (thickness 0.3048)))
     )
@@
     (at 51 74.5 180)
     (descr "SMD LED, 1206")
-    (fp_text reference D1 (at 0 -1.651 180) (layer F.SilkS)
+    (fp_text reference D1 (at 0.0222 -1.6746 180) (layer F.SilkS)
       (effects (font (size 0.8001 0.8001) (thickness 0.14986)))
     )
-    (fp_text value LED (at 0 1.80086 180) (layer F.SilkS)
+    (fp_text value LED (at -0.054 1.602 180) (layer F.SilkS)
       (effects (font (size 0.8001 0.8001) (thickness 0.14986)))
     )
@@
       (effects (font (size 0.8001 0.8001) (thickness 0.14986)))
     )
-    (fp_text value LED (at 0 1.80086 180) (layer F.SilkS)
+    (fp_text value LED (at -0.023 1.7962 180) (layer F.SilkS)
       (effects (font (size 0.8001 0.8001) (thickness 0.14986)))
     )
@@
     (at 51 70.5 180)
     (descr "SMT resistor, 1210")
-    (fp_text reference R1 (at 0 -1.7526 180) (layer F.SilkS)
+    (fp_text reference R1 (at -0.0286 -0.0612 180) (layer F.SilkS)
       (effects (font (size 0.50038 0.50038) (thickness 0.11938)))
     )
@@
     (at 88.8 70.6 180)
     (descr "SMT resistor, 1210")
-    (fp_text reference R2 (at 0 -1.7526 180) (layer F.SilkS)
+    (fp_text reference R2 (at -0.0238 0.0134 180) (layer F.SilkS)
       (effects (font (size 0.50038 0.50038) (thickness 0.11938)))
     )
@@
     (at 88.9 67.3 180)
     (descr "SMT resistor, 1210")
-    (fp_text reference R3 (at 0 -1.7526 180) (layer F.SilkS)
+    (fp_text reference R3 (at 0.0762 -0.0608 180) (layer F.SilkS)
       (effects (font (size 0.50038 0.50038) (thickness 0.11938)))
     )
@@
       (effects (font (size 1 1) (thickness 0.15)))
     )
-    (fp_text value 3.5mmM3 (at 0 -0.5) (layer F.Fab)
+    (fp_text value 3.5mmM3 (at 0 -0.5) (layer F.Fab) hide
       (effects (font (size 1 1) (thickness 0.15)))
     )
@@
       (effects (font (size 1 1) (thickness 0.15)))
     )
-    (fp_text value 3.5mmM3 (at 0 -0.5) (layer F.Fab)
+    (fp_text value 3.5mmM3 (at 0 -0.5) (layer F.Fab) hide
       (effects (font (size 1 1) (thickness 0.15)))
     )
@@
       (effects (font (size 1 1) (thickness 0.15)))
     )
-    (fp_text value 3.5mmM3 (at 0 -0.5) (layer F.Fab)
+    (fp_text value 3.5mmM3 (at 0 -0.5) (layer F.Fab) hide
       (effects (font (size 1 1) (thickness 0.15)))
     )
@@
       (effects (font (size 1 1) (thickness 0.15)))
     )
-    (fp_text value 3.5mmM3 (at 0 -0.5) (layer F.Fab)
+    (fp_text value 3.5mmM3 (at 0 -0.5) (layer F.Fab) hide
       (effects (font (size 1 1) (thickness 0.15)))
     )
@@
       (effects (font (size 1 1) (thickness 0.15)))
     )
-    (fp_text value JUMPER (at 5.08 3.81 180) (layer F.Fab)
+    (fp_text value JUMPER (at 5.08 3.81 180) (layer F.Fab) hide
       (effects (font (size 1 1) (thickness 0.15)))
     )
@@
     (descr "Terminal block 3 pins")
     (tags DEV)
-    (fp_text reference P7 (at 0 -5.842 270) (layer F.SilkS)
+    (fp_text reference P7 (at 0 -5.842 270) (layer F.SilkS) hide
       (effects (font (thickness 0.3048)))
     )
@@
     )
   )
+  (gr_circle (center 88.215 81.4122) (end 87.515 80.7872) (layer B.SilkS) (width 0.2))
+  (gr_text R (at 88.165 81.4872) (layer B.SilkS)
+    (effects (font (size 0.8 0.8) (thickness 0.2)) (justify mirror))
+  )
+  (gr_text G (at 72.1136 81.3102) (layer B.SilkS)
+    (effects (font (size 0.8 0.8) (thickness 0.2)) (justify mirror))
+  )
+  (gr_circle (center 72.0636 81.3352) (end 71.3636 80.7102) (layer B.SilkS) (width 0.2))
+  (gr_text L (at 76.8418 81.08) (layer B.SilkS)
+    (effects (font (size 0.8 0.8) (thickness 0.2)) (justify mirror))
+  )
+  (gr_circle (center 76.8918 81.205) (end 76.1918 80.58) (layer B.SilkS) (width 0.2))
+  (gr_circle (center 82.928 81.4094) (end 82.228 80.7844) (layer B.SilkS) (width 0.2))
+  (gr_text G (at 82.878 81.4094) (layer B.SilkS)
+    (effects (font (size 0.8 0.8) (thickness 0.2)) (justify mirror))
+  )
   (gr_text +5V (at 60.35 47.95) (layer B.SilkS)
